File: AnalogFadingLED/HysteresisOscillator/AnalogFaderV2/AnalogFaderV2.kicad_pcb (KiCad board)
At the start: 2 copper layers, 45.8 x 19.1 mm, 45 parts, among them J1 Conn_01x06_Female, J2 Conn_01x06_Female, J3 USB_B_Micro, SW1 SW_DIP_x03, U1 LMV358

Commit message: Added V2 files
Other:
- board text added: "Analog Fader V2.0"
